Commit message: add ikfast for VP-6242G

File: vp6242_description/urdf/vp6242.urdf (robot description, URDF)
Before this commit: robot vp6242, 9 links, 8 joints
Links:
- removed link base
- added link world
Joints:
- removed joint base-base_link
- added joint fixed: type fixed, parent world, child base_link
- joint joint6: axis 1 0 0 -> 0 0 1; origin xyz=0.0 0.0 0.07 rpy=0 -1.570796 0 -> xyz=0.0 0.0 0.07 rpy=0 0 0

File: vp6242_description/urdf/vp6242_macro.xacro (robot description, xacro)
@@ -44,4 +44,7 @@
                 </geometry>
                 <xacro:mesh_origin/>
+                <material name="blue">
+					<color rgba="0 0 1 1"/>
+				</material>
             </visual>
             <collision>
@@ -50,4 +53,7 @@
         	  	</geometry>
                 <xacro:mesh_origin/>
+                <material name="yellow">
+					<color rgba="0 1 1 1"/>
+				</material>
             </collision>
             <inertial>
@@ -190,6 +196,6 @@
             <axis xyz="0 0 1"/>
             <limit
+                lower="${joint1_min}"
                 upper="${joint1_max}"
-                lower="${joint1_min}"
                 effort="${default_joint_effort}"
                 velocity="${default_joint_velocity}" />
@@ -202,6 +208,6 @@
             <axis xyz="0 1 0"/>
             <limit
+                lower="${joint2_min}"
                 upper="${joint2_max}"
-                lower="${joint2_min}"
                 effort="${default_joint_effort}"
                 velocity="${default_joint_velocity}" />
@@ -214,6 +220,6 @@
             <axis xyz="0 1 0"/>
             <limit
+                lower="${joint3_min}"
                 upper="${joint3_max}"
-                lower="${joint3_min}"
                 effort="${default_joint_effort}"
                 velocity="${default_joint_velocity}"/>
@@ -226,6 +232,6 @@
             <axis xyz="0 0 1"/>
             <limit
+                lower="${joint4_min}"
                 upper="${joint4_max}"
-                lower="${joint4_min}"
                 effort="${default_joint_effort}"
                 velocity="${default_joint_velocity}"/>
@@ -238,6 +244,6 @@
             <axis xyz="0 1 0"/>
             <limit
+                lower="${joint5_min}"
                 upper="${joint5_max}"
-                lower="${joint5_min}"
                 effort="${default_joint_effort}"
                 velocity="${default_joint_velocity}"/>
@@ -250,6 +256,6 @@
             <axis xyz="0 0 1"/>
             <limit
+                lower="${joint6_min}"
                 upper="${joint6_max}"
-                lower="${joint6_min}"
                 effort="${default_joint_effort}"
                 velocity="${default_joint_velocity}"/>

Commit message: add moveit and ikfast for VP6242

File: vp6242_description/urdf/vp6242.urdf (robot description, URDF)
Before this commit: robot vp6242, 9 links, 8 joints
Joints:
- removed joint fixed
- added joint world-base: type fixed, parent world, child base_link

File: vp6242_description/urdf/vp6242_macro.xacro (robot description, xacro)
@@ -36,5 +36,5 @@
     <xacro:macro name="vp6242" params="prefix">
  <!-- Used for fixing robot to Gazebo 'base_link' -->
-        <link name="world"/>
+        <link name="${prefix}world"/>
         <link name="${prefix}base_link">
             <xacro:default_inertial mass="10"/>
@@ -186,7 +186,7 @@
         <link name="${prefix}tool0"/>
         <!-- Joint list -->
-        <joint name="fixed" type="fixed">
-             <parent link="world"/>
-             <child link="${prefix}base_link"/>
+        <joint name="${prefix}world-base" type="fixed">
+            <parent link="${prefix}world"/>
+            <child link="${prefix}base_link"/>
         </joint>
         <joint name="${prefix}joint1" type="revolute">
