Commit message: Migrated to new xacro version. Fixed transmission control issues.

File: vp6242_description/urdf/vp6242.xacro (robot description, xacro)
@@ -1,5 +1,6 @@
 <?xml version="1.0" ?>
-<robot name="vp6242" xmlns:xacro="http://ros.org/wiki/xacro">
-	<include filename="$(find vp6242_description)/urdf/vp6242_macro.xacro"/>
+<!-- <robot name="vp6242" xmlns:xacro="http://ros.org/wiki/xacro"> -->
+<robot name="vp6242" xmlns:xacro="http://www.ros.org/wiki/xacro">
+	<xacro:include filename="$(find vp6242_description)/urdf/vp6242_macro.xacro"/>
 	<xacro:vp6242 prefix=""/>
 </robot>

File: vp6242_description/urdf/vp6242_macro.xacro (robot description, xacro)
@@ -35,24 +35,30 @@
     </gazebo>
     <gazebo reference="${prefix}link1">
+      <material>Gazebo/Red</material>
       <gravity>false</gravity>
       <selfCollide>false</selfCollide>
     </gazebo>
     <gazebo reference="${prefix}link2">
+      <material>Gazebo/Green</material>
       <gravity>false</gravity>
       <selfCollide>false</selfCollide>
     </gazebo>
     <gazebo reference="${prefix}link3">
+      <material>Gazebo/Orange</material>
       <gravity>false</gravity>
       <selfCollide>false</selfCollide>
     </gazebo>
     <gazebo reference="${prefix}link4">
+      <material>Gazebo/Indigo</material>
       <gravity>false</gravity>
       <selfCollide>false</selfCollide>
     </gazebo>
     <gazebo reference="${prefix}link5">
+      <material>Gazebo/Purple</material>
       <gravity>false</gravity>
       <selfCollide>false</selfCollide>
     </gazebo>
     <gazebo reference="${prefix}link6">
+      <material>Gazebo/Yellow</material>
       <gravity>false</gravity>
       <selfCollide>false</selfCollide>
@@ -261,4 +267,5 @@
       <origin xyz="0 0 0" rpy="0 0 0"/>
     </joint>
+    <!--
     <transmission name="${prefix}tran1" type="transmission_interface/SimpleTransmission">
       <joint name="${prefix}joint1"/>
@@ -266,26 +273,50 @@
       <mechanicalReduction>1</mechanicalReduction>
     </transmission>
-    <transmission name="${prefix}tran2" type="transmission_interface/SimpleTransmission">
-      <joint name="${prefix}joint2"/>
+    !-->
+    <transmission name="${prefix}tran1">
+      <type>transmission_interface/SimpleTransmission</type>
+      <joint name="${prefix}joint1">
+        <hardwareInterface>hardware_interface/EffortJointInterface</hardwareInterface>
+      </joint>
+      <actuator name="${prefix}motor1" type="EffortJointInterface" />
+      <mechanicalReduction>1</mechanicalReduction>
+    </transmission>
+    <transmission name="${prefix}tran2">
+      <type>transmission_interface/SimpleTransmission</type>
+      <joint name="${prefix}joint2">
+        <hardwareInterface>hardware_interface/EffortJointInterface</hardwareInterface>
+      </joint>
       <actuator name="${prefix}motor2" type="EffortJointInterface" />
       <mechanicalReduction>1</mechanicalReduction>
     </transmission>
-    <transmission name="${prefix}tran3" type="transmission_interface/SimpleTransmission">
-      <joint name="${prefix}joint3"/>
+    <transmission name="${prefix}tran3">
+      <type>transmission_interface/SimpleTransmission</type>
+      <joint name="${prefix}joint3">
+        <hardwareInterface>hardware_interface/EffortJointInterface</hardwareInterface>
+      </joint>
       <actuator name="${prefix}motor3" type="EffortJointInterface" />
       <mechanicalReduction>1</mechanicalReduction>
     </transmission>
-    <transmission name="${prefix}tran4" type="transmission_interface/SimpleTransmission">
-      <joint name="${prefix}joint4"/>
+    <transmission name="${prefix}tran4">
+      <type>transmission_interface/SimpleTransmission</type>
+      <joint name="${prefix}joint4">
+        <hardwareInterface>hardware_interface/EffortJointInterface</hardwareInterface>
+      </joint>
       <actuator name="${prefix}motor4" type="EffortJointInterface" />
       <mechanicalReduction>1</mechanicalReduction>
     </transmission>
-    <transmission name="${prefix}tran5" type="transmission_interface/SimpleTransmission">
-      <joint name="${prefix}joint5"/>
+    <transmission name="${prefix}tran5">
+      <type>transmission_interface/SimpleTransmission</type>
+      <joint name="${prefix}joint5">
+        <hardwareInterface>hardware_interface/EffortJointInterface</hardwareInterface>
+      </joint>
       <actuator name="${prefix}motor5" type="EffortJointInterface" />
       <mechanicalReduction>1</mechanicalReduction>
     </transmission>
-    <transmission name="${prefix}tran6" type="transmission_interface/SimpleTransmission">
-      <joint name="${prefix}joint6"/>
+    <transmission name="${prefix}tran6">
+      <type>transmission_interface/SimpleTransmission</type>
+      <joint name="${prefix}joint6">
+        <hardwareInterface>hardware_interface/EffortJointInterface</hardwareInterface>
+      </joint>
       <actuator name="${prefix}motor6" type="EffortJointInterface" />
       <mechanicalReduction>1</mechanicalReduction>
