Commit message: Setando os ângulos iguais ao Denso do lab

File: vp6242_description/urdf/vp6242_macro.xacro (robot description, xacro)
@@ -1,271 +1,265 @@
-<?xml version="1.0"?>
+<?xml version="1.0" encoding="UTF-8"?>
 <robot xmlns:xacro="http://www.ros.org/wiki/xacro">
-  <!-- Limits Joint: J1 J2 J3 J4 J5 J6
+   <!-- Limits Joint: J1 J2 J3 J4 J5 J6
                Max : 160 120 160 160 120 360
                Min :-160 -120 19 -160 -120 -360 -->
-  <xacro:macro name="mesh_origin">
-    <origin rpy="-1.570796 3.141592 0" xyz="0 0 0"/>
-  </xacro:macro>
-  <xacro:property name="mesh_path" value="package://vp6242_description/meshes" />
-  <xacro:property name="mesh_scale" value="0.001 0.001 0.001" />
-  <xacro:property name="default_joint_velocity" value="0.8" />
-  <xacro:property name="default_joint_effort" value="25000" />
-  <xacro:property name="joint1_min" value="-2.792526803"/>
-  <xacro:property name="joint1_max" value="2.792526803"/>
-  <xacro:property name="joint2_min" value="-2.094395102"/>
-  <xacro:property name="joint2_max" value="2.094395102"/>
-  <xacro:property name="joint3_min" value="0.331612558"/>
-  <xacro:property name="joint3_max" value="2.792526803"/>
-  <xacro:property name="joint4_min" value="-2.792526803"/>
-  <xacro:property name="joint4_max" value="2.792526803"/>
-  <xacro:property name="joint5_min" value="-2.094395102"/>
-  <xacro:property name="joint5_max" value="2.094395102"/>
-  <xacro:property name="joint6_min" value="-6.283185307"/>
-  <xacro:property name="joint6_max" value="6.283185307"/>
-  <gazebo>
-    <plugin name="ros_control" filename="libgazebo_ros_control.so">
-      <robotNamespace>/vp6242</robotNamespace>
-    </plugin>
-  </gazebo>
-  <xacro:macro name="vp6242" params="prefix">
-    <gazebo reference="${prefix}base_link">
-      <material>Gazebo/Blue</material>
-      <gravity>false</gravity>
-      <selfCollide>false</selfCollide>
-    </gazebo>
-    <gazebo reference="${prefix}link1">
-      <material>Gazebo/Red</material>
-      <gravity>false</gravity>
-      <selfCollide>false</selfCollide>
-    </gazebo>
-    <gazebo reference="${prefix}link2">
-      <material>Gazebo/Green</material>
-      <gravity>false</gravity>
-      <selfCollide>false</selfCollide>
-    </gazebo>
-    <gazebo reference="${prefix}link3">
-      <material>Gazebo/Orange</material>
-      <gravity>false</gravity>
-      <selfCollide>false</selfCollide>
-    </gazebo>
-    <gazebo reference="${prefix}link4">
-      <material>Gazebo/Indigo</material>
-      <gravity>false</gravity>
-      <selfCollide>false</selfCollide>
-    </gazebo>
-    <gazebo reference="${prefix}link5">
-      <material>Gazebo/Purple</material>
-      <gravity>false</gravity>
-      <selfCollide>false</selfCollide>
-    </gazebo>
-    <gazebo reference="${prefix}link6">
-      <material>Gazebo/Yellow</material>
-      <gravity>false</gravity>
-      <selfCollide>false</selfCollide>
-    </gazebo>
-    <!-- Used for fixing robot to Gazebo 'base_link' -->
-    <link name="${prefix}world"/>
-    <link name="${prefix}base_link">
-      <visual>
-        <geometry>
-          <mesh filename="${mesh_path}/visual/base.dae" scale="${mesh_scale}"/>
-        </geometry>
-        <xacro:mesh_origin/>
-      </visual>
-      <collision>
-        <geometry>
-          <mesh filename="${mesh_path}/collision/base.dae" scale="${mesh_scale}"/>
-        </geometry>
-        <xacro:mesh_origin/>
-      </collision>
-      <inertial>
-        <origin xyz="0 0 0.0775" rpy="0 0 0"/>
-        <mass value="1"/>
-        <inertia  ixx="1.0" ixy="0.0" ixz="0.0" iyy="1.0" iyz="0.0" izz="1.0"/>
-      </inertial>
-    </link>
-    <link name="${prefix}link1">
-      <visual>
-        <geometry>
-          <mesh filename="${mesh_path}/visual/link1.dae" scale="${mesh_scale}"/>
-        </geometry>
-        <xacro:mesh_origin/>
-      </visual>
-      <collision>
-        <geometry>
-          <mesh filename="${mesh_path}/collision/link1.dae" scale="${mesh_scale}"/>
-        </geometry>
-        <xacro:mesh_origin/>
-      </collision>
-      <inertial>
-        <origin xyz="0 0 0.0625" rpy="0 0 0"/>
-        <mass value="1"/>
-        <inertia  ixx="1.0" ixy="0.0" ixz="0.0" iyy="1.0" iyz="0.0" izz="1.0"/>
-      </inertial>
-    </link>
-    <link name="${prefix}link2">
-      <visual>
-        <geometry>
-          <mesh filename="${mesh_path}/visual/link2.dae" scale="${mesh_scale}"/>
-        </geometry>
-        <xacro:mesh_origin/>
-      </visual>
-      <collision>
-        <geometry>
-          <mesh filename="${mesh_path}/collision/link2.dae" scale="${mesh_scale}"/>
-        </geometry>
-        <xacro:mesh_origin/>
-      </collision>
-      <inertial>
-        <origin xyz="0 0 0.105" rpy="0 0 0"/>
-        <mass value="1"/>
-        <inertia  ixx="1.0" ixy="0.0" ixz="0.0" iyy="1.0" iyz="0.0" izz="1.0"/>
-      </inertial>
-    </link>
-    <link name="${prefix}link3">
-      <visual>
-        <geometry>
-          <mesh filename="${mesh_path}/visual/link3.dae" scale="${mesh_scale}"/>
-        </geometry>
-        <origin rpy="-1.570796 1.570796 0" xyz="0 0 0"/>
-      </visual>
-      <collision>
-        <geometry>
-          <mesh filename="${mesh_path}/collision/link3.dae" scale="${mesh_scale}"/>
-        </geometry>
-        <origin rpy="-1.570796 1.570796 0" xyz="0 0 0"/>
-      </collision>
-      <inertial>
-        <origin xyz="-0.075 0 0" rpy="0 0 0"/>
-        <mass value="1"/>
-        <inertia  ixx="1.0" ixy="0.0" ixz="0.0" iyy="1.0" iyz="0.0" izz="1.0"/>
-      </inertial>
-    </link>
-    <link name="${prefix}link4">
-      <visual>
-        <geometry>
-          <mesh filename="${mesh_path}/visual/link4.dae" scale="${mesh_scale}"/>
-        </geometry>
-        <origin rpy="0 1.570796 1.570796" xyz="0 0 0.085"/>
-      </visual>
-      <collision>
-        <geometry>
-          <mesh filename="${mesh_path}/collision/link4.dae" scale="${mesh_scale}"/>
-        </geometry>
-        <origin rpy="0 1.570796 1.570796" xyz="0 0 0.085"/>
-      </collision>
-       <inertial>
-        <origin xyz="0 0 0.13" rpy="0 0 0"/>
-        <mass value="1"/>
-        <inertia  ixx="1.0" ixy="0.0" ixz="0.0" iyy="1.0" iyz="0.0" izz="1.0"/>
-      </inertial>
-    </link>
-    <link name="${prefix}link5">
-      <visual>
-        <geometry>
-          <mesh filename="${mesh_path}/visual/link5.dae" scale="${mesh_scale}"/>
-        </geometry>
-        <origin rpy="0 1.570796 1.570796" xyz="0 0 0.0"/>
-      </visual>
-      <collision>
-        <geometry>
-          <mesh filename="${mesh_path}/collision/link5.dae" scale="${mesh_scale}"/>
-        </geometry>
-        <origin rpy="0 1.570796 1.570796" xyz="0 0 0.0"/>
-      </collision>
-      <inertial>
-        <origin xyz="0 0 0" rpy="0 0 0"/>
-        <mass value="1"/>
-        <inertia  ixx="1.0" ixy="0.0" ixz="0.0"  iyy="1.0" iyz="0.0"  izz="1.0"/>
-      </inertial>
-    </link>
-    <link name="${prefix}link6">
-      <visual>
-        <geometry>
-          <cylinder length="0.01" radius="0.0205"/>
-        </geometry>
-        <origin rpy="0 0 0" xyz="0.0 0.0 -0.005"/>
-        <material name="plate">
-          <color rgba="0.1 0.1 0.1 0.8"/>
-        </material>
-      </visual>
-      <collision>
-        <geometry>
-          <cylinder length="0.01" radius="0.0205"/>
-        </geometry>
-        <origin rpy="0 0 0" xyz="0.0 0.0 -0.005"/>
-      </collision>
-      <inertial>
-        <origin xyz="0 0 0" rpy="0 0 0"/>
-        <mass value="0.2"/>
-        <inertia  ixx="1.0" ixy="0.0" ixz="0.0"  iyy="1.0" iyz="0.0"  izz="1.0"/>
-      </inertial>
-    </link>
-    <link name="${prefix}tool0"/>
-    <!-- Joint list -->
-    <joint name="${prefix}world-base" type="fixed">
-      <parent link="${prefix}world"/>
-      <child link="${prefix}base_link"/>
-    </joint>
-    <joint name="${prefix}joint1" type="revolute">
-      <origin rpy="0 0 0" xyz="0.0 0.0 0.155"/>
-      <parent link="${prefix}base_link"/>
-      <child link="${prefix}link1"/>
-      <axis xyz="0 0 1"/>
-      <limit  lower="${joint1_min}"  upper="${joint1_max}"  effort="${default_joint_effort}"
-        velocity="${default_joint_velocity}" />
-      <dynamics damping="0.7"/>
-    </joint>
-    <joint name="${prefix}joint2" type="revolute">
-      <origin rpy="0 0 0" xyz="0.0 0.0 0.125"/>
-      <parent link="${prefix}link1"/>
-      <child link="${prefix}link2"/>
-      <axis xyz="0 1 0"/>
-      <limit  lower="${joint2_min}"  upper="${joint2_max}"  effort="${default_joint_effort}"
-        velocity="${default_joint_velocity}" />
-      <dynamics damping="0.7"/>
-    </joint>
-    <joint name="${prefix}joint3" type="revolute">
-      <origin rpy="0 0 0" xyz="0.0 0.0 0.210"/>
-      <parent link="${prefix}link2"/>
-      <child link="${prefix}link3"/>
-      <axis xyz="0 1 0"/>
-      <limit  lower="${joint3_min}"  upper="${joint3_max}"  effort="${default_joint_effort}"
-        velocity="${default_joint_velocity}"/>
-      <dynamics damping="0.7"/>
-    </joint>
-    <joint name="${prefix}joint4" type="revolute">
-      <origin rpy="0 0 0" xyz="-0.075 0.0 0.0"/>
-      <parent link="${prefix}link3"/>
-      <child link="${prefix}link4"/>
-      <axis xyz="0 0 1"/>
-      <limit  lower="${joint4_min}"  upper="${joint4_max}"  effort="${default_joint_effort}"
-        velocity="${default_joint_velocity}"/>
-      <dynamics damping="0.7"/>
-    </joint>
-    <joint name="${prefix}joint5" type="revolute">
-      <origin rpy="0 0 0" xyz="0.0 0.0 0.210"/>
-      <parent link="${prefix}link4"/>
-      <child link="${prefix}link5"/>
-      <axis xyz="0 1 0"/>
-      <limit lower="${joint5_min}"  upper="${joint5_max}"  effort="${default_joint_effort}"
-        velocity="${default_joint_velocity}"/>
-      <dynamics damping="0.7"/>
-    </joint>
-    <joint name="${prefix}joint6" type="revolute">
-      <origin rpy="0 0 0" xyz="0.0 0.0 0.07"/>
-      <parent link="${prefix}link5"/>
-      <child link="${prefix}link6"/>
-      <axis xyz="0 0 1"/>
-      <limit  lower="${joint6_min}"  upper="${joint6_max}"  effort="${default_joint_effort}"
-        velocity="${default_joint_velocity}"/>
-      <dynamics damping="0.7"/>
-    </joint>
-    <joint name="${prefix}joint6-tool0" type="fixed">
-      <parent link="${prefix}link6"/>
-      <child link="${prefix}tool0"/>
-      <origin xyz="0 0 0" rpy="0 0 0"/>
-    </joint>
-    <!--
+   <xacro:macro name="mesh_origin">
+      <origin rpy="-1.570796 3.141592 0" xyz="0 0 0" />
+   </xacro:macro>
+   <xacro:property name="mesh_path" value="package://vp6242_description/meshes" />
+   <xacro:property name="mesh_scale" value="0.001 0.001 0.001" />
+   <xacro:property name="default_joint_velocity" value="0.8" />
+   <xacro:property name="default_joint_effort" value="25000" />
+   <xacro:property name="joint1_min" value="-2.792526803" />
+   <xacro:property name="joint1_max" value="2.792526803" />
+   <xacro:property name="joint2_min" value="-2.094395102" />
+   <xacro:property name="joint2_max" value="2.094395102" />
+   <xacro:property name="joint3_min" value="-2.792526803" />
+   <xacro:property name="joint3_max" value="2.792526803" />
+   <xacro:property name="joint4_min" value="-2.792526803" />
+   <xacro:property name="joint4_max" value="2.792526803" />
+   <xacro:property name="joint5_min" value="-2.094395102" />
+   <xacro:property name="joint5_max" value="2.094395102" />
+   <xacro:property name="joint6_min" value="-6.283185307" />
+   <xacro:property name="joint6_max" value="6.283185307" />
+   <gazebo>
+      <plugin name="ros_control" filename="libgazebo_ros_control.so">
+         <robotNamespace>/vp6242</robotNamespace>
+      </plugin>
+   </gazebo>
+   <xacro:macro name="vp6242" params="prefix">
+      <gazebo reference="${prefix}base_link">
+         <material>Gazebo/Blue</material>
+         <gravity>false</gravity>
+         <selfCollide>false</selfCollide>
+      </gazebo>
+      <gazebo reference="${prefix}link1">
+         <material>Gazebo/Red</material>
+         <gravity>false</gravity>
+         <selfCollide>false</selfCollide>
+      </gazebo>
+      <gazebo reference="${prefix}link2">
+         <material>Gazebo/Green</material>
+         <gravity>false</gravity>
+         <selfCollide>false</selfCollide>
+      </gazebo>
+      <gazebo reference="${prefix}link3">
+         <material>Gazebo/Orange</material>
+         <gravity>false</gravity>
+         <selfCollide>false</selfCollide>
+      </gazebo>
+      <gazebo reference="${prefix}link4">
+         <material>Gazebo/Indigo</material>
+         <gravity>false</gravity>
+         <selfCollide>false</selfCollide>
+      </gazebo>
+      <gazebo reference="${prefix}link5">
+         <material>Gazebo/Purple</material>
+         <gravity>false</gravity>
+         <selfCollide>false</selfCollide>
+      </gazebo>
+      <gazebo reference="${prefix}link6">
+         <material>Gazebo/Yellow</material>
+         <gravity>false</gravity>
+         <selfCollide>false</selfCollide>
+      </gazebo>
+      <!-- Used for fixing robot to Gazebo 'base_link' -->
+      <link name="${prefix}world" />
+      <link name="${prefix}base_link">
+         <visual>
+            <geometry>
+               <mesh filename="${mesh_path}/visual/base.dae" scale="${mesh_scale}" />
+            </geometry>
+            <xacro:mesh_origin />
+         </visual>
+         <collision>
+            <geometry>
+               <mesh filename="${mesh_path}/collision/base.dae" scale="${mesh_scale}" />
+            </geometry>
+            <xacro:mesh_origin />
+         </collision>
+         <inertial>
+            <origin xyz="0 0 0.0775" rpy="0 0 0" />
+            <mass value="1" />
+            <inertia ixx="1.0" ixy="0.0" ixz="0.0" iyy="1.0" iyz="0.0" izz="1.0" />
+         </inertial>
+      </link>
+      <link name="${prefix}link1">
+         <visual>
+            <geometry>
+               <mesh filename="${mesh_path}/visual/link1.dae" scale="${mesh_scale}" />
+            </geometry>
+            <xacro:mesh_origin />
+         </visual>
+         <collision>
+            <geometry>
+               <mesh filename="${mesh_path}/collision/link1.dae" scale="${mesh_scale}" />
+            </geometry>
+            <xacro:mesh_origin />
+         </collision>
+         <inertial>
+            <origin xyz="0 0 0.0625" rpy="0 0 0" />
+            <mass value="1" />
+            <inertia ixx="1.0" ixy="0.0" ixz="0.0" iyy="1.0" iyz="0.0" izz="1.0" />
+         </inertial>
+      </link>
+      <link name="${prefix}link2">
+         <visual>
+            <geometry>
+               <mesh filename="${mesh_path}/visual/link2.dae" scale="${mesh_scale}" />
+            </geometry>
+            <xacro:mesh_origin />
+         </visual>
+         <collision>
+            <geometry>
+               <mesh filename="${mesh_path}/collision/link2.dae" scale="${mesh_scale}" />
+            </geometry>
+            <xacro:mesh_origin />
+         </collision>
+         <inertial>
+            <origin xyz="0 0 0.105" rpy="0 0 0" />
+            <mass value="1" />
+            <inertia ixx="1.0" ixy="0.0" ixz="0.0" iyy="1.0" iyz="0.0" izz="1.0" />
+         </inertial>
+      </link>
+      <link name="${prefix}link3">
+         <visual>
+            <geometry>
+               <mesh filename="${mesh_path}/visual/link3.dae" scale="${mesh_scale}" />
+            </geometry>
+            <origin rpy="-1.570796 1.570796 0" xyz="0 0 0" />
+         </visual>
+         <collision>
+            <geometry>
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