Commit message: change name to match with ROS style

File: hg_agv_description/urdf/hg_agv_macro.xacro (robot description, xacro)
@@ -7,7 +7,7 @@
     <origin rpy="0 0 0" xyz="0 0 0"/>
   </xacro:macro>
-  <xacro:property name="mesh_path" value="package://hg-agv_description/meshes" />
+  <xacro:property name="mesh_path" value="package://hg_agv_description/meshes" />
   <xacro:property name="mesh_scale" value="0.001 0.001 0.001" />
-  <xacro:macro name="hg-agv" params="prefix">
+  <xacro:macro name="hg_agv" params="prefix">
     <link name="${prefix}mobile_base"/>
     <link name="${prefix}base_link">

Commit message: add swivel

File: hg_agv_description/urdf/hg_agv_macro.xacro (robot description, xacro)
@@ -25,7 +25,8 @@
       </collision>
       <inertial>
-        <origin xyz="0 0 0" rpy="0 0 0"/>
-        <mass value="5"/>
-        <inertia  ixx="1.0" ixy="0.0" ixz="0.0" iyy="1.0" iyz="0.0" izz="1.0"/>
+        <origin xyz="-0.091316 0 0.184078" rpy="0 0 0"/>
+        <mass value="23.911"/>
+        <inertia  ixx="5.748" ixy="3.453" ixz="0.413"
+                  iyy="6.144" iyz="0.002" izz="1.131"/>
       </inertial>
     </link>
@@ -49,7 +50,8 @@
       </collision>
       <inertial>
-        <origin xyz="0 0 0" rpy="0 0 0"/>
-        <mass value="1"/>
-        <inertia  ixx="1.0" ixy="0.0" ixz="0.0" iyy="1.0" iyz="0.0" izz="1.0"/>
+        <mass value="1.031"/>
+        <origin xyz="0 0.015293 0"/>
+          <inertia ixx="0.005" ixy="0" ixz="0"
+                   iyy="0.007" iyz="0" izz="0.005"/>
       </inertial>
     </link>
@@ -74,7 +76,8 @@
       </collision>
       <inertial>
-        <origin xyz="0 0 0" rpy="0 0 0"/>
-        <mass value="1"/>
-        <inertia  ixx="1.0" ixy="0.0" ixz="0.0" iyy="1.0" iyz="0.0" izz="1.0"/>
+        <mass value="1.031"/>
+        <origin xyz="0 -0.015293 0"/>
+          <inertia ixx="0.005" ixy="0" ixz="0"
+                   iyy="0.007" iyz="0" izz="0.005"/>
       </inertial>
     </link>
@@ -85,48 +88,94 @@
       <child link="${prefix}right_wheel"/>
     </joint>
-    <link name="${prefix}urg04lx">
+    <link name="${prefix}left_swivel_base">
       <visual>
         <geometry>
-          <mesh filename="${mesh_path}/urg04lx.dae" scale="${mesh_scale}"/>
+          <mesh filename="${mesh_path}/swivel_base.dae" scale="${mesh_scale}"/>
+        </geometry>
+        <origin rpy="0 0 0" xyz="0 0 -0.01"/>
+      </visual>
+    </link>
+    <joint name="${prefix}base_left_swivel_base" type="fixed">
+      <origin rpy="0 0 0" xyz="-0.605 0.12 -0.012"/>
+      <parent link="${prefix}base_link"/>
+      <child link="${prefix}left_swivel_base"/>
+    </joint>
+    <link name="${prefix}left_swivel_cover">
+      <visual>
+        <geometry>
+          <mesh filename="${mesh_path}/swivel_cover.dae" scale="${mesh_scale}"/>
+        </geometry>
+        <origin rpy="0 0 0" xyz="-0.033 0 -0.054"/>
+      </visual>
+    </link>
+    <joint name="${prefix}left_swivel_base_cover" type="continuous">
+      <axis xyz="0 0 1"/>
+      <origin rpy="0 0 0" xyz="0 0 -0.01"/>
+      <parent link="${prefix}left_swivel_base"/>
+      <child link="${prefix}left_swivel_cover"/>
+    </joint>
+    <link name="${prefix}left_swivel_wheel">
+      <visual>
+        <geometry>
+          <mesh filename="${mesh_path}/swivel_wheel.dae" scale="${mesh_scale}"/>
         </geometry>
         <xacro:mesh_origin/>
       </visual>
-      <collision>
+    </link>
+    <joint name="${prefix}left_swivel_cover_wheel" type="continuous">
+      <axis xyz="0 1 0"/>
+      <origin rpy="0 0 0" xyz="-0.033 0 -0.054"/>
+      <parent link="${prefix}left_swivel_cover"/>
+      <child link="${prefix}left_swivel_wheel"/>
+    </joint>
+    <link name="${prefix}right_swivel_base">
+      <visual>
         <geometry>
-          <mesh filename="${mesh_path}/urg04lx_collision.dae" scale="${mesh_scale}"/>
+          <mesh filename="${mesh_path}/swivel_base.dae" scale="${mesh_scale}"/>
+        </geometry>
+        <origin rpy="0 0 0" xyz="0 0 -0.01"/>
+      </visual>
+    </link>
+    <joint name="${prefix}base_right_swivel_base" type="fixed">
+      <origin rpy="0 0 0" xyz="-0.605 -0.12 -0.012"/>
+      <parent link="${prefix}base_link"/>
+      <child link="${prefix}right_swivel_base"/>
+    </joint>
+    <link name="${prefix}right_swivel_cover">
+      <visual>
+        <geometry>
+          <mesh filename="${mesh_path}/swivel_cover.dae" scale="${mesh_scale}"/>
+        </geometry>
+        <origin rpy="0 0 0" xyz="-0.033 0 -0.054"/>
+      </visual>
+    </link>
+    <joint name="${prefix}right_swivel_base_cover" type="continuous">
+      <axis xyz="0 0 1"/>
+      <origin rpy="0 0 0" xyz="0 0 -0.01"/>
+      <parent link="${prefix}right_swivel_base"/>
+      <child link="${prefix}right_swivel_cover"/>
+    </joint>
+    <link name="${prefix}right_swivel_wheel">
+      <visual>
+        <geometry>
+          <mesh filename="${mesh_path}/swivel_wheel.dae" scale="${mesh_scale}"/>
         </geometry>
         <xacro:mesh_origin/>
-      </collision>
-      <inertial>
-        <origin xyz="0 0 0" rpy="0 0 0"/>
-        <mass value="1"/>
-        <inertia  ixx="1.0" ixy="0.0" ixz="0.0" iyy="1.0" iyz="0.0" izz="1.0"/>
-      </inertial>
+      </visual>
     </link>
-    <joint name="${prefix}base-urg40lx" type="fixed">
+    <joint name="${prefix}right_swivel_cover_wheel" type="continuous">
+      <axis xyz="0 1 0"/>
+      <origin rpy="0 0 0" xyz="-0.033 0 -0.054"/>
+      <parent link="${prefix}right_swivel_cover"/>
+      <child link="${prefix}right_swivel_wheel"/>
+    </joint>
+    <link name="${prefix}urg04lx"/>
+    <joint name="${prefix}base_urg40lx" type="fixed">
       <origin rpy="0 0 0" xyz="0.08 0 0.134"/>
       <parent link="${prefix}base_link"/>
       <child link="${prefix}urg04lx"/>
     </joint>
-    <link name="${prefix}utm30lx">
-      <visual>
-        <geometry>
-          <mesh filename="${mesh_path}/utm30lx.dae" scale="${mesh_scale}"/>
-        </geometry>
-        <xacro:mesh_origin/>
-      </visual>
-      <collision>
-        <geometry>
-          <mesh filename="${mesh_path}/utm30lx_collision.dae" scale="${mesh_scale}"/>
-        </geometry>
-        <xacro:mesh_origin/>
-      </collision>
-      <inertial>
-        <origin xyz="0 0 0" rpy="0 0 0"/>
-        <mass value="1"/>
-        <inertia  ixx="1.0" ixy="0.0" ixz="0.0" iyy="1.0" iyz="0.0" izz="1.0"/>
-      </inertial>
-    </link>
-    <joint name="${prefix}base-utm30lx" type="fixed">
+    <link name="${prefix}utm30lx"/>
+    <joint name="${prefix}base_utm30lx" type="fixed">
       <origin rpy="0 0 0" xyz="-0.1805 0 1.914"/>
       <parent link="${prefix}base_link"/>

Commit message: update xacro

File: hg_agv_description/urdf/hg_agv_macro.xacro (robot description, xacro)
@@ -9,4 +9,89 @@
   <xacro:property name="mesh_path" value="package://hg_agv_description/meshes" />
   <xacro:property name="mesh_scale" value="0.001 0.001 0.001" />
+  <xacro:property name="pi" value="3.141592" />
+  <xacro:macro name="swivel" params="side reflect">
+    <link name="${prefix}${side}_swivel_base">
+      <visual>
+        <geometry>
+          <mesh filename="${mesh_path}/swivel_base.dae" scale="${mesh_scale}"/>
+        </geometry>
+        <origin rpy="0 0 0" xyz="0 0 -0.01"/>
+      </visual>
+    </link>
+    <joint name="${prefix}base_${side}_swivel_base" type="fixed">
+      <origin rpy="0 0 0" xyz="-0.6045 ${reflect*0.12} -0.012"/>
+      <parent link="${prefix}base_link"/>
+      <child link="${prefix}${side}_swivel_base"/>
+    </joint>
+    <link name="${prefix}${side}_swivel_cover">
+      <visual>
+        <geometry>
+          <mesh filename="${mesh_path}/swivel_cover.dae" scale="${mesh_scale}"/>
+        </geometry>
+        <origin rpy="0 0 0" xyz="-0.033 0 -0.054"/>
+      </visual>
+    </link>
+    <joint name="${prefix}${side}_swivel_base_cover" type="continuous">
+      <axis xyz="0 0 1"/>
+      <origin rpy="0 0 0" xyz="0 0 -0.01"/>
+      <parent link="${prefix}${side}_swivel_base"/>
+      <child link="${prefix}${side}_swivel_cover"/>
+    </joint>
+    <link name="${prefix}${side}_swivel_wheel">
+      <visual>
+        <geometry>
+          <mesh filename="${mesh_path}/swivel_wheel.dae" scale="${mesh_scale}"/>
+        </geometry>
+        <xacro:mesh_origin/>
+      </visual>
+      <!--collision>
+        <geometry>
+          <cylinder length="0.02" radius="0.038"/>
+        </geometry>
+        <origin rpy="${pi/2} 0 0" xyz="0 0 0"/>
+      </collision-->
+    </link>
+    <joint name="${prefix}${side}_swivel_cover_wheel" type="continuous">
+      <axis xyz="0 1 0"/>
+      <origin rpy="0 0 0" xyz="-0.033 0 -0.054"/>
+      <parent link="${prefix}${side}_swivel_cover"/>
+      <child link="${prefix}${side}_swivel_wheel"/>
+    </joint>
+  </xacro:macro>
+  <xacro:macro name="wheel" params="side reflect flip">
+    <link name="${prefix}${side}_wheel">
+      <visual>
+        <geometry>
+          <mesh filename="${mesh_path}/wheel.dae" scale="${mesh_scale}"/>
+        </geometry>
+        <origin rpy="0 0 ${flip*pi}" xyz="0 0 0"/>
+      </visual>
+      <collision>
+        <geometry>
+          <mesh filename="${mesh_path}/wheel_collision.dae" scale="${mesh_scale}"/>
+        </geometry>
+        <origin rpy="0 0 ${flip*pi}" xyz="0 0 0"/>
+      </collision>
+      <!--inertial>
+        <mass value="1.031"/>
+        <origin xyz="0 ${reflect*0.015293} 0"/>
+          <inertia ixx="0.005" ixy="0" ixz="0"
+                   iyy="0.007" iyz="0" izz="0.005"/>
+      </inertial-->
+      <inertial>
+        <origin xyz="0 0 0" rpy="0 0 0"/>
+        <mass value="1"/>
+        <inertia  ixx="1.0" ixy="0.0" ixz="0.0"
+                  iyy="1.0" iyz="0.0"
+                  izz="1.0"/>
+      </inertial>
+    </link>
+    <joint name="${prefix}${side}_wheel_joint" type="continuous">
+      <axis xyz="0 1 0"/>
+      <origin rpy="0 0 0" xyz="0 ${reflect*0.1956} 0"/>
+      <parent link="${prefix}base_link"/>
+      <child link="${prefix}${side}_wheel"/>
+    </joint>
+  </xacro:macro>
   <xacro:macro name="hg_agv" params="prefix">
     <link name="${prefix}mobile_base"/>
@@ -24,9 +109,16 @@
         <xacro:mesh_origin/>
       </collision>
-      <inertial>
+      <!--inertial>
         <origin xyz="-0.091316 0 0.184078" rpy="0 0 0"/>
         <mass value="23.911"/>
         <inertia  ixx="5.748" ixy="3.453" ixz="0.413"
                   iyy="6.144" iyz="0.002" izz="1.131"/>
+      </inertial-->
+      <inertial>
+        <origin xyz="0 0 0" rpy="0 0 0"/>
+        <mass value="1"/>
+        <inertia  ixx="1.0" ixy="0.0" ixz="0.0"
+                  iyy="1.0" iyz="0.0"
+                  izz="1.0"/>
       </inertial>
     </link>
@@ -36,138 +128,8 @@
       <child link="${prefix}base_link"/>
     </joint>
-    <link name="${prefix}left_wheel">
-      <visual>
-        <geometry>
-          <mesh filename="${mesh_path}/left_wheel.dae" scale="${mesh_scale}"/>
-        </geometry>
-        <xacro:mesh_origin/>
-      </visual>
-      <collision>
-        <geometry>
-          <mesh filename="${mesh_path}/left_wheel_collision.dae" scale="${mesh_scale}"/>
-        </geometry>
-        <xacro:mesh_origin/>
-      </collision>
-      <inertial>
-        <mass value="1.031"/>
-        <origin xyz="0 0.015293 0"/>
-          <inertia ixx="0.005" ixy="0" ixz="0"
-                   iyy="0.007" iyz="0" izz="0.005"/>
-      </inertial>
-    </link>
-    <joint name="${prefix}left_wheel_joint" type="continuous">
-      <axis xyz="0 1 0"/>
-      <origin rpy="0 0 0" xyz="0 0.1956 0"/>
-      <parent link="${prefix}base_link"/>
-      <child link="${prefix}left_wheel"/>
-    </joint>
-    <link name="${prefix}right_wheel">
-      <visual>
-        <geometry>
-          <mesh filename="${mesh_path}/right_wheel.dae" scale="${mesh_scale}"/>
-        </geometry>
-        <xacro:mesh_origin/>
-      </visual>
-      <collision>
-        <geometry>
-          <mesh filename="${mesh_path}/right_wheel_collision.dae" scale="${mesh_scale}"/>
-        </geometry>
-        <xacro:mesh_origin/>
-      </collision>
-      <inertial>
-        <mass value="1.031"/>
-        <origin xyz="0 -0.015293 0"/>
-          <inertia ixx="0.005" ixy="0" ixz="0"
-                   iyy="0.007" iyz="0" izz="0.005"/>
-      </inertial>
-    </link>
-    <joint name="${prefix}right_wheel_joint" type="continuous">
-      <axis xyz="0 1 0"/>
-      <origin rpy="0 0 0" xyz="0 -0.1956 0"/>
-      <parent link="${prefix}base_link"/>
-      <child link="${prefix}right_wheel"/>
-    </joint>
-    <link name="${prefix}left_swivel_base">
-      <visual>
-        <geometry>
-          <mesh filename="${mesh_path}/swivel_base.dae" scale="${mesh_scale}"/>
-        </geometry>
-        <origin rpy="0 0 0" xyz="0 0 -0.01"/>
-      </visual>
-    </link>
-    <joint name="${prefix}base_left_swivel_base" type="fixed">
-      <origin rpy="0 0 0" xyz="-0.605 0.12 -0.012"/>
-      <parent link="${prefix}base_link"/>
-      <child link="${prefix}left_swivel_base"/>
-    </joint>
-    <link name="${prefix}left_swivel_cover">
-      <visual>
-        <geometry>
-          <mesh filename="${mesh_path}/swivel_cover.dae" scale="${mesh_scale}"/>
-        </geometry>
-        <origin rpy="0 0 0" xyz="-0.033 0 -0.054"/>
-      </visual>
-    </link>
-    <joint name="${prefix}left_swivel_base_cover" type="continuous">
-      <axis xyz="0 0 1"/>
-      <origin rpy="0 0 0" xyz="0 0 -0.01"/>
-      <parent link="${prefix}left_swivel_base"/>
-      <child link="${prefix}left_swivel_cover"/>
-    </joint>
-    <link name="${prefix}left_swivel_wheel">
-      <visual>
-        <geometry>
-          <mesh filename="${mesh_path}/swivel_wheel.dae" scale="${mesh_scale}"/>
-        </geometry>
-        <xacro:mesh_origin/>
-      </visual>
-    </link>
-    <joint name="${prefix}left_swivel_cover_wheel" type="continuous">
-      <axis xyz="0 1 0"/>
-      <origin rpy="0 0 0" xyz="-0.033 0 -0.054"/>
-      <parent link="${prefix}left_swivel_cover"/>
-      <child link="${prefix}left_swivel_wheel"/>
-    </joint>
-    <link name="${prefix}right_swivel_base">
-      <visual>
-        <geometry>
-          <mesh filename="${mesh_path}/swivel_base.dae" scale="${mesh_scale}"/>
-        </geometry>
-        <origin rpy="0 0 0" xyz="0 0 -0.01"/>
-      </visual>
-    </link>
-    <joint name="${prefix}base_right_swivel_base" type="fixed">
-      <origin rpy="0 0 0" xyz="-0.605 -0.12 -0.012"/>
-      <parent link="${prefix}base_link"/>
-      <child link="${prefix}right_swivel_base"/>
-    </joint>
-    <link name="${prefix}right_swivel_cover">
-      <visual>
-        <geometry>
-          <mesh filename="${mesh_path}/swivel_cover.dae" scale="${mesh_scale}"/>
-        </geometry>
-        <origin rpy="0 0 0" xyz="-0.033 0 -0.054"/>
-      </visual>
-    </link>
-    <joint name="${prefix}right_swivel_base_cover" type="continuous">
-      <axis xyz="0 0 1"/>
-      <origin rpy="0 0 0" xyz="0 0 -0.01"/>
-      <parent link="${prefix}right_swivel_base"/>
-      <child link="${prefix}right_swivel_cover"/>
-    </joint>
-    <link name="${prefix}right_swivel_wheel">
-      <visual>
-        <geometry>
-          <mesh filename="${mesh_path}/swivel_wheel.dae" scale="${mesh_scale}"/>
-        </geometry>
-        <xacro:mesh_origin/>
-      </visual>
-    </link>
-    <joint name="${prefix}right_swivel_cover_wheel" type="continuous">
-      <axis xyz="0 1 0"/>
-      <origin rpy="0 0 0" xyz="-0.033 0 -0.054"/>
-      <parent link="${prefix}right_swivel_cover"/>
-      <child link="${prefix}right_swivel_wheel"/>
-    </joint>
+    <xacro:wheel side="left" reflect="1" flip="0"/>
+    <xacro:wheel side="right" reflect="-1" flip="1"/>
+    <xacro:swivel side="left" reflect="1" />
+    <xacro:swivel side="right" reflect="-1" />
     <link name="${prefix}urg04lx"/>
     <joint name="${prefix}base_urg40lx" type="fixed">
