Commit message: add LRF

File: hg_agv_description/urdf/hg_agv_macro.xacro (robot description, xacro)
@@ -4,4 +4,6 @@
                Max : 160 120 160 160 120 360
                Min :-160 -120 19 -160 -120 -360 -->
+  <!-- Import Rviz colors -->
+  <xacro:include filename="$(find hg_agv_description)/urdf/materials.xacro" />
   <xacro:macro name="mesh_origin">
     <origin rpy="0 0 0" xyz="0 0 0"/>
@@ -10,4 +12,10 @@
   <xacro:property name="mesh_scale" value="0.001 0.001 0.001" />
   <xacro:property name="pi" value="3.141592" />
+  <!-- ros_control plugin -->
+  <gazebo>
+    <plugin name="ros_control" filename="libgazebo_ros_control.so">
+      <robotNamespace>/hg_agv</robotNamespace>
+    </plugin>
+  </gazebo>
   <xacro:macro name="swivel" params="side reflect">
     <link name="${prefix}${side}_swivel_base">
@@ -18,68 +26,13 @@
         <origin rpy="0 0 0" xyz="0 0 -0.01"/>
       </visual>
-    </link>
-    <joint name="${prefix}base_${side}_swivel_base" type="fixed">
-      <origin rpy="0 0 0" xyz="-0.6045 ${reflect*0.12} -0.012"/>
-      <parent link="${prefix}base_link"/>
-      <child link="${prefix}${side}_swivel_base"/>
-    </joint>
-    <link name="${prefix}${side}_swivel_cover">
-      <visual>
-        <geometry>
-          <mesh filename="${mesh_path}/swivel_cover.dae" scale="${mesh_scale}"/>
-        </geometry>
-        <origin rpy="0 0 0" xyz="-0.033 0 -0.054"/>
-      </visual>
-    </link>
-    <joint name="${prefix}${side}_swivel_base_cover" type="continuous">
-      <axis xyz="0 0 1"/>
-      <origin rpy="0 0 0" xyz="0 0 -0.01"/>
-      <parent link="${prefix}${side}_swivel_base"/>
-      <child link="${prefix}${side}_swivel_cover"/>
-    </joint>
-    <link name="${prefix}${side}_swivel_wheel">
-      <visual>
-        <geometry>
-          <mesh filename="${mesh_path}/swivel_wheel.dae" scale="${mesh_scale}"/>
-        </geometry>
-        <xacro:mesh_origin/>
-      </visual>
-      <!--collision>
-        <geometry>
-          <cylinder length="0.02" radius="0.038"/>
-        </geometry>
-        <origin rpy="${pi/2} 0 0" xyz="0 0 0"/>
-      </collision-->
-    </link>
-    <joint name="${prefix}${side}_swivel_cover_wheel" type="continuous">
-      <axis xyz="0 1 0"/>
-      <origin rpy="0 0 0" xyz="-0.033 0 -0.054"/>
-      <parent link="${prefix}${side}_swivel_cover"/>
-      <child link="${prefix}${side}_swivel_wheel"/>
-    </joint>
-  </xacro:macro>
-  <xacro:macro name="wheel" params="side reflect flip">
-    <link name="${prefix}${side}_wheel">
-      <visual>
-        <geometry>
-          <mesh filename="${mesh_path}/wheel.dae" scale="${mesh_scale}"/>
-        </geometry>
-        <origin rpy="0 0 ${flip*pi}" xyz="0 0 0"/>
-      </visual>
-      <collision>
-        <geometry>
-          <mesh filename="${mesh_path}/wheel_collision.dae" scale="${mesh_scale}"/>
-        </geometry>
-        <origin rpy="0 0 ${flip*pi}" xyz="0 0 0"/>
-      </collision>
-      <!--inertial>
-        <mass value="1.031"/>
-        <origin xyz="0 ${reflect*0.015293} 0"/>
-          <inertia ixx="0.005" ixy="0" ixz="0"
-                   iyy="0.007" iyz="0" izz="0.005"/>
-      </inertial-->
+      <collision>
+        <geometry>
+          <box size="0 0 0"/>
+        </geometry>
+        <origin rpy="0 0 0" xyz="0 0 0"/>
+      </collision>
       <inertial>
         <origin xyz="0 0 0" rpy="0 0 0"/>
-        <mass value="1"/>
+        <mass value="0.01"/>
         <inertia  ixx="1.0" ixy="0.0" ixz="0.0"
                   iyy="1.0" iyz="0.0"
@@ -87,10 +40,114 @@
       </inertial>
     </link>
+    <joint name="${prefix}base_${side}_swivel_base_joint" type="fixed">
+      <origin rpy="0 0 0" xyz="-0.6045 ${reflect*0.12} -0.012"/>
+      <parent link="${prefix}base_link"/>
+      <child link="${prefix}${side}_swivel_base"/>
+    </joint>
+    <link name="${prefix}${side}_swivel_cover">
+      <visual>
+        <geometry>
+          <mesh filename="${mesh_path}/swivel_cover.dae" scale="${mesh_scale}"/>
+        </geometry>
+        <origin rpy="0 0 0" xyz="-0.033 0 -0.054"/>
+      </visual>
+      <collision>
+        <geometry>
+          <box size="0 0 0"/>
+        </geometry>
+        <origin rpy="0 0 0" xyz="0 0 0"/>
+      </collision>
+      <inertial>
+        <origin xyz="0 0 0" rpy="0 0 0"/>
+        <mass value="0.01"/>
+        <inertia  ixx="1.0" ixy="0.0" ixz="0.0"
+                  iyy="1.0" iyz="0.0"
+                  izz="1.0"/>
+      </inertial>
+    </link>
+    <joint name="${prefix}${side}_swivel_base_cover_joint" type="continuous">
+      <axis xyz="0 0 1"/>
+      <origin rpy="0 0 0" xyz="0 0 -0.01"/>
+      <limit effort="100" velocity="100" k_velocity="0" />
+    	<joint_properties damping="0.0" friction="0.0" />
+      <parent link="${prefix}${side}_swivel_base"/>
+      <child link="${prefix}${side}_swivel_cover"/>
+    </joint>
+    <link name="${prefix}${side}_swivel_wheel">
+      <visual>
+        <geometry>
+          <mesh filename="${mesh_path}/swivel_wheel.dae" scale="${mesh_scale}"/>
+        </geometry>
+        <xacro:mesh_origin/>
+      </visual>
+      <collision>
+        <geometry>
+          <mesh filename="${mesh_path}/swivel_wheel_collision.dae" scale="${mesh_scale}"/>
+        </geometry>
+        <xacro:mesh_origin/>
+      </collision>
+      <inertial>
+        <origin xyz="0 0 0" rpy="0 0 0"/>
+        <mass value="0.1"/>
+        <inertia  ixx="1.0" ixy="0.0" ixz="0.0"
+                  iyy="1.0" iyz="0.0"
+                  izz="1.0"/>
+      </inertial>
+    </link>
+    <joint name="${prefix}${side}_swivel_cover_wheel_joint" type="continuous">
+      <axis xyz="0 1 0"/>
+      <origin rpy="0 0 0" xyz="-0.033 0 -0.054"/>
+      <limit effort="100" velocity="100" k_velocity="0" />
+    	<joint_properties damping="0.0" friction="0.0" />
+      <parent link="${prefix}${side}_swivel_cover"/>
+      <child link="${prefix}${side}_swivel_wheel"/>
+    </joint>
+    <gazebo reference="${prefix}${side}_swivel_wheel">
+      <mu1>0.2</mu1>
+      <mu2>0.2</mu2>
+      <material>Gazebo/Black</material>
+    </gazebo>
+  </xacro:macro>
+  <xacro:macro name="wheel" params="side reflect flip">
+    <link name="${prefix}${side}_wheel">
+      <visual>
+        <geometry>
+          <mesh filename="${mesh_path}/wheel.dae" scale="${mesh_scale}"/>
+        </geometry>
+        <origin rpy="0 0 ${flip*pi}" xyz="0 0 0"/>
+        <material name="black"/>
+      </visual>
+      <collision>
+        <geometry>
+          <mesh filename="${mesh_path}/wheel_collision.dae" scale="${mesh_scale}"/>
+        </geometry>
+        <origin rpy="0 0 ${flip*pi}" xyz="0 0 0"/>
+      </collision>
+      <inertial>
+        <origin xyz="0 ${reflect*0.015293} 0"/>
+        <mass value="1"/>
+        <inertia
+          ixx="1.0" ixy="0.0" ixz="0.0"
+          iyy="1.0" iyz="0.0"
+          izz="1.0"/>
+        <!--mass value="1.031"/>
+        <inertia ixx="0.005" ixy="0" ixz="0"
+                 iyy="0.007" iyz="0"
+                 izz="0.005"/-->
+      </inertial>
+    </link>
     <joint name="${prefix}${side}_wheel_joint" type="continuous">
       <axis xyz="0 1 0"/>
       <origin rpy="0 0 0" xyz="0 ${reflect*0.1956} 0"/>
+      <limit effort="100" velocity="100" />
+      <dynamics damping="0.7"/>
       <parent link="${prefix}base_link"/>
       <child link="${prefix}${side}_wheel"/>
     </joint>
+    <gazebo reference="${prefix}${side}_wheel">
+      <mu1>0.2</mu1>
+      <mu2>0.2</mu2>
+      <material>Gazebo/Black</material>
+    </gazebo>
   </xacro:macro>
   <xacro:macro name="hg_agv" params="prefix">
@@ -109,16 +166,16 @@
         <xacro:mesh_origin/>
       </collision>
-      <!--inertial>
+      <inertial>
         <origin xyz="-0.091316 0 0.184078" rpy="0 0 0"/>
+        <!--mass value="1"/>
+        <inertia
+          ixx="1.0" ixy="0.0" ixz="0.0"
+          iyy="1.0" iyz="0.0"
+          izz="1.0"/-->
         <mass value="23.911"/>
-        <inertia  ixx="5.748" ixy="3.453" ixz="0.413"
-                  iyy="6.144" iyz="0.002" izz="1.131"/>
-      </inertial-->
-      <inertial>
-        <origin xyz="0 0 0" rpy="0 0 0"/>
-        <mass value="1"/>
-        <inertia  ixx="1.0" ixy="0.0" ixz="0.0"
-                  iyy="1.0" iyz="0.0"
-                  izz="1.0"/>
+        <inertia
+          ixx="5.748" ixy="3.453" ixz="0.413"
+          iyy="6.144" iyz="0.002"
+          izz="1.131"/>
       </inertial>
     </link>
@@ -132,16 +189,86 @@
     <xacro:swivel side="left" reflect="1" />
     <xacro:swivel side="right" reflect="-1" />
-    <link name="${prefix}urg04lx"/>
-    <joint name="${prefix}base_urg40lx" type="fixed">
-      <origin rpy="0 0 0" xyz="0.08 0 0.134"/>
-      <parent link="${prefix}base_link"/>
-      <child link="${prefix}urg04lx"/>
-    </joint>
-    <link name="${prefix}utm30lx"/>
-    <joint name="${prefix}base_utm30lx" type="fixed">
-      <origin rpy="0 0 0" xyz="-0.1805 0 1.914"/>
-      <parent link="${prefix}base_link"/>
-      <child link="${prefix}utm30lx"/>
-    </joint>
+    <link name="${prefix}laser_button"/>
+    <joint name="${prefix}laser_button_joint" type="fixed">
+      <origin rpy="0 0 0" xyz="0.08 0 0.194"/>
+      <parent link="${prefix}base_link"/>
+      <child link="${prefix}laser_button"/>
+    </joint>
+    <link name="${prefix}laser_top"/>
+    <joint name="${prefix}laser_top_joint" type="fixed">
+      <origin rpy="0 0 0" xyz="-0.1805 0 1.974"/>
+      <parent link="${prefix}base_link"/>
+      <child link="${prefix}laser_top"/>
+    </joint>
+    <gazebo reference="${prefix}laser_button">
+      <sensor type="gpu_ray" name="button_hokuyo_sensor">
+        <pose>0 0 0 0 0 0</pose>
+        <visualize>true</visualize>
+        <update_rate>40</update_rate>
+        <ray>
+          <scan>
+            <horizontal>
+              <samples>682</samples>
+              <resolution>1</resolution>
+              <min_angle>-2.09439</min_angle>
+              <max_angle>2.09439</max_angle>
+            </horizontal>
+          </scan>
+          <range>
+            <min>0.1</min>
+            <max>4.095</max>
+            <resolution>0.03</resolution>
+          </range>
+          <noise>
+            <type>gaussian</type>
+            <!-- Noise parameters based on published spec for Hokuyo laser
+                 achieving "+-30mm" accuracy at range < 10m.  A mean of 0.0m and
+                 stddev of 0.01m will put 99.7% of samples within 0.03m of the true
+                 reading. -->
+            <mean>0.0</mean>
+            <stddev>0.01</stddev>
+          </noise>
+        </ray>
+        <plugin name="button_hokuyo_sensor_controller" filename="libgazebo_ros_gpu_laser.so">
+          <topicName>/hg_agv/laser_buttom/scan</topicName>
+          <frameName>laser_button</frameName>
+        </plugin>
+      </sensor>
+    </gazebo>
+    <gazebo reference="${prefix}laser_top">
+      <sensor type="gpu_ray" name="top_hokuyo_sensor">
+        <pose>0 0 0 0 0 0</pose>
+        <visualize>true</visualize>
+        <update_rate>40</update_rate>
+        <ray>
+          <scan>
+            <horizontal>
+              <samples>1080</samples>
+              <resolution>1</resolution>
+              <min_angle>-2.35619</min_angle>
+              <max_angle>2.35619</max_angle>
+            </horizontal>
+          </scan>
+          <range>
+            <min>0.1</min>
+            <max>30.0</max>
+            <resolution>0.01</resolution>
+          </range>
+          <noise>
+            <type>gaussian</type>
+            <!-- Noise parameters based on published spec for Hokuyo laser
+                 achieving "+-30mm" accuracy at range < 10m.  A mean of 0.0m and
+                 stddev of 0.01m will put 99.7% of samples within 0.03m of the true
+                 reading. -->
+            <mean>0.0</mean>
+            <stddev>0.01</stddev>
+          </noise>
+        </ray>
+        <plugin name="top_hokuyo_sensor_controller" filename="libgazebo_ros_gpu_laser.so">
+          <topicName>/hg_agv/laser_top/scan</topicName>
+          <frameName>laser_top</frameName>
+        </plugin>
+      </sensor>
+    </gazebo>
   </xacro:macro>
 </robot>
